File: kicad/stepper_analyzer.kicad_pcb (KiCad board)
At the start: 2 copper layers, 102 x 57 mm, 24 parts, among them J1 Connector_Conn_01x04_Male, J2 Connector_Conn_01x04_Male, M1 Motor, Q1 AO3400A, U1 ACS70331EOLCTR-2P5B3, U2 ACS70331EOLCTR-2P5B3, U3 Pico

Commit message: Remove orhpan text message.
Other:
- board text removed: "IMPORTANT: Apply here 0.2mm thick double sided tape to avoid shroting the TFT and the PCB."

Commit message: Updated label on the PCB.
Other:
- board text added: "CAPACITIVE TOUCH FT6206 I2C BOTTOM CONTACTS"
- board text removed: "CAPACITIVE TOUCH FT6236 I2C BOTTOM CONTACTS"
