File: kicad/stepper_analyzer.sch (KiCad schematic (older format))
At the start: 23 parts, among them J1 Connector_Conn_01x04_Male, J2 Connector_Conn_01x04_Male, M1 Motor, Q1 AO3400A, U1 ACS70331EOLCTR-2P5B3, U2 ACS70331EOLCTR-2P5B3, U3 Pico

Commit message: Renamed Config to Options
Parts:
- R4, R5: footprint stepper_motor_analyzer:R_0805_2012Metric_Pad1.15x1.40mm_HandSolder -> stepper_motor_analyzer:R_0805_2012Metric_Pad1.15x1.40mm_HandSolder_no_3d
Connections:
- net CONFIG renamed OPTIONS
Changed lines of the file:
@@
 	3500 6550 2800 6550
 Text Label 2800 6550 0    50   ~ 0
-CONFIG
+OPTIONS
 Text Notes 1550 6950 0    50   ~ 0
 RESERVED FOR\nFUTURE\nFEATURES
@@
 F 0 "R4" H 1150 6800 50  0000 L CNN
 F 1 "DNP" H 1150 6900 50  0000 L CNN
-F 2 "stepper_motor_analyzer:R_0805_2012Metric_Pad1.15x1.40mm_HandSolder" V 1390 6840 50  0001 C CNN
+F 2 "stepper_motor_analyzer:R_0805_2012Metric_Pad1.15x1.40mm_HandSolder_no_3d" V 1390 6840 50  0001 C CNN
 F 3 "~" H 1350 6850 50  0001 C CNN
 F 4 "" V 1350 6850 50  0001 C CNN "LCSC"
@@
 F 0 "R5" H 1450 6500 50  0000 L CNN
 F 1 "DNP" H 1400 6400 50  0000 L CNN
-F 2 "stepper_motor_analyzer:R_0805_2012Metric_Pad1.15x1.40mm_HandSolder" V 1390 6440 50  0001 C CNN
+F 2 "stepper_motor_analyzer:R_0805_2012Metric_Pad1.15x1.40mm_HandSolder_no_3d" V 1390 6440 50  0001 C CNN
 F 3 "~" H 1350 6450 50  0001 C CNN
 F 4 "" V 1350 6450 50  0001 C CNN "LCSC"
@@
 	1350 6650 1350 6700
 Text Label 1800 6650 2    50   ~ 0
-CONFIG
+OPTIONS
 Wire Wire Line
 	5150 5950 5150 6450

Commit message: Made schematic and PCB changes toward MK3.  Not ready.
Parts:
- added C4, C5: DNP, stepper_motor_analyzer:C_0805_2012Metric_Pad1.15x1.40mm_HandSolder, symbol Device:C
Connections:
- net +3V3: no longer FPC1.12 (Pin_12)
- net GND: now also U3.27 (GP21), C4.1, C5.1
- net ~TFT_RD: now reaches U3.29 (GP22)
- net ~TFT_RD: now also FPC1.12 (Pin_12)
- net at U2.6 (NC): now also C5.2
- net at U1.6 (NC): now also C4.2
- no-connect marks 20 -> 18
Other:
- note added: "(MK4)"
- note added: "Simple Stepper Motor Analyzer MK4"
- note added: "WORK IN PROGRESS. NON RELEASE."
- note removed: "Simple Stepper Motor Analyzer MK2"
Changed lines of the file:
@@
 L power:GND #PWR0105
 U 1 1 60A1DF96
-P 3850 2050
-F 0 "#PWR0105" H 3850 1800 50  0001 C CNN
-F 1 "GND" H 3855 1877 50  0000 C CNN
-F 2 "" H 3850 2050 50  0001 C CNN
-F 3 "" H 3850 2050 50  0001 C CNN
-	1    3850 2050
-	1    0    0    -1
-$EndComp
-Wire Wire Line
-	3850 2000 3850 2050
+P 3850 2100
+F 0 "#PWR0105" H 3850 1850 50  0001 C CNN
+F 1 "GND" H 3855 1927 50  0000 C CNN
+F 2 "" H 3850 2100 50  0001 C CNN
+F 3 "" H 3850 2100 50  0001 C CNN
+	1    3850 2100
+	1    0    0    -1
+$EndComp
+Wire Wire Line
+	3850 2000 3850 2100
 Text Label 4750 1500 2    50   ~ 0
 CHB
@@
 L power:GND #PWR0108
 U 1 1 60A49E54
-P 2900 3150
-F 0 "#PWR0108" H 2900 2900 50  0001 C CNN
-F 1 "GND" H 2905 2977 50  0000 C CNN
-F 2 "" H 2900 3150 50  0001 C CNN
-F 3 "" H 2900 3150 50  0001 C CNN
-	1    2900 3150
-	1    0    0    -1
-$EndComp
-Wire Wire Line
-	2900 3150 2900 3100
+P 2900 3200
+F 0 "#PWR0108" H 2900 2950 50  0001 C CNN
+F 1 "GND" H 2905 3027 50  0000 C CNN
+F 2 "" H 2900 3200 50  0001 C CNN
+F 3 "" H 2900 3200 50  0001 C CNN
+	1    2900 3200
+	1    0    0    -1
+$EndComp
 Wire Wire Line
 	2900 2300 2900 2150
@@
 ~TFT_WR
 Wire Wire Line
-	8500 2450 8900 2450
-Wire Wire Line
 	8500 1450 8500 1850
 NoConn ~ 8900 2650
@@
 Connection ~ 8700 2150
 Connection ~ 8700 2850
-Connection ~ 8500 2450
 Wire Wire Line
 	8900 4950 8700 4950
@@
 Connection ~ 8500 1950
 Wire Wire Line
-	8500 1950 8500 2450
-Wire Wire Line
 	8900 5250 8700 5250
 Connection ~ 8700 5250
 Wire Wire Line
 	8700 5250 8700 5800
-Wire Wire Line
-	8500 2450 8500 4550
 $Comp
 L power:GND #PWR0120
@@
 $EndComp
 Text Notes 6400 7150 0    100  ~ 0
-Simple Stepper Motor Analyzer MK2
+Simple Stepper Motor Analyzer MK4
 Text Notes 7550 4850 2    50   ~ 0
 BACKLIGHT\nCONTROL
@@
 Wire Wire Line
 	8700 4450 8700 4950
-NoConn ~ 4900 6050
 NoConn ~ 4900 6150
 NoConn ~ 4900 6250
@@
 NoConn ~ 4900 6650
 NoConn ~ 3500 5150
-NoConn ~ 4900 5750
 $Comp
 L Transistor_FET:AO3400A Q1
@@
 Text Label 2800 4850 0    50   ~ 0
 ~TFT_RST
-NoConn ~ 4900 5850
 $Comp
 L Device:C C3
@@
 OPTIONS
 Wire Wire Line
-	5150 5950 5150 6450
+	5150 5950 5150 6050
 NoConn ~ 4900 6350
+Text Label 5650 5850 2    50   ~ 0
+~TFT_RD
+Wire Wire Line
+	8500 1950 8500 4550
+Wire Wire Line
+	8900 2450 8050 2450
+Text Label 8050 2450 0    50   ~ 0
+~TFT_RD
+Wire Wire Line
+	4900 5850 5650 5850
+NoConn ~ 4900 5750
+$Comp
+L Device:C C5
+U 1 1 60ECCB29
+P 4350 1900
+F 0 "C5" H 4150 1900 50  0000 L CNN
+F 1 "DNP" H 4100 2000 50  0000 L CNN
+F 2 "stepper_motor_analyzer:C_0805_2012Metric_Pad1.15x1.40mm_HandSolder" H 4388 1750 50  0001 C CNN
+F 3 "~" H 4350 1900 50  0001 C CNN
+F 4 "C49678 " V 4350 1900 50  0001 C CNN "LCSC"
+	1    4350 1900
+	-1   0    0    1
+$EndComp
+$Comp
+L power:GND #PWR0111
+U 1 1 60ECD31D
+P 4350 2100
+F 0 "#PWR0111" H 4350 1850 50  0001 C CNN
+F 1 "GND" H 4355 1927 50  0000 C CNN
+F 2 "" H 4350 2100 50  0001 C CNN
+F 3 "" H 4350 2100 50  0001 C CNN
+	1    4350 2100
+	1    0    0    -1
+$EndComp
+Wire Wire Line
+	4300 1700 4350 1700
+Wire Wire Line
+	4350 1700 4350 1750
+Wire Wire Line
+	4350 2050 4350 2100
+$Comp
+L Device:C C4
+U 1 1 60EE9FA1
+P 3400 3000
+F 0 "C4" H 3200 3000 50  0000 L CNN
+F 1 "DNP" H 3150 3100 50  0000 L CNN
+F 2 "stepper_motor_analyzer:C_0805_2012Metric_Pad1.15x1.40mm_HandSolder" H 3438 2850 50  0001 C CNN
+F 3 "~" H 3400 3000 50  0001 C CNN
+F 4 "C49678 " V 3400 3000 50  0001 C CNN "LCSC"
+	1    3400 3000
+	-1   0    0    1
+$EndComp
+$Comp
+L power:GND #PWR0112
+U 1 1 60EEA675
+P 3400 3200
+F 0 "#PWR0112" H 3400 2950 50  0001 C CNN
+F 1 "GND" H 3405 3027 50  0000 C CNN
+F 2 "" H 3400 3200 50  0001 C CNN
+F 3 "" H 3400 3200 50  0001 C CNN
+	1    3400 3200
+	1    0    0    -1
+$EndComp
+Wire Wire Line
+	3350 2800 3400 2800
+Wire Wire Line
+	3400 2800 3400 2850
+Wire Wire Line
+	3400 3150 3400 3200
+Wire Wire Line
+	2900 3100 2900 3200
+Text Notes 4650 1950 0    50   ~ 0
+(MK4)
+Text Notes 3700 3050 0    50   ~ 0
+(MK4)
+Text Notes 5700 5850 0    50   ~ 0
+(MK4)
+Wire Wire Line
+	4900 6050 5150 6050
+Connection ~ 5150 6050
+Wire Wire Line
+	5150 6050 5150 6450
+Text Notes 4900 6050 0    50   ~ 0
+(MK4)
+Text Notes 6400 6950 0    100  ~ 0
+WORK IN PROGRESS. NON RELEASE.
 $EndSCHEMATC

Commit message: Teaked board design toward MK4.
Parts:
- C4: value DNP -> 1nf
- R4: footprint stepper_motor_analyzer:R_0805_2012Metric_Pad1.15x1.40mm_HandSolder_no_3d -> stepper_motor_analyzer:R_0805_2012Metric_Pad1.15x1.40mm_HandSolder
- U1, U2: value ACS70331EOLCTR-2P5B3 -> (CURRENT SENSOR)
Other:
- note added: "1K"
- note added: "1nf"
- note added: "ACS70331EOLCTR-2P5B3"
- note added: "ACS712ELCTR-05B-T"
- note added: "C4, C5"
- note added: "CONFIG"
- note added: "DNP"
- note added: "R4"
- note added: "R5"
- note added: "SENSOR"
- moved on the sheet: C3, R4, R5, TP3, U3

Commit message: Assorted tweaks.
Parts:
- added R? (x3): 1K, stepper_motor_analyzer:R_0805_2012Metric_Pad1.15x1.40mm_HandSolder, symbol Device:R_US
- added R?: DNP, stepper_motor_analyzer:R_0805_2012Metric_Pad1.15x1.40mm_HandSolder, symbol Device:R_US
Connections:
- net labels added: +5V
- wire segments 165 -> 173
- no-connect marks 18 -> 17
Other:
- note added: "WORK IN PROGRESS. USE RELEASE INSTEAD"
- note removed: "WORK IN PROGRESS. NON RELEASE."
- moved on the sheet: C1, C2, C4, C5, J1, J2, U1, U2

Commit message: Made the shcematic non-release warning more visible.
Parts:
- gave numbers to parts that had none: 4
Changed lines of the file:
@@
 Text Notes 3450 3450 0    50   ~ 0
 (MK4)
-Text Notes 6400 6950 0    100  ~ 0
+Text Notes 1250 4400 0    236  ~ 47
 WORK IN PROGRESS. USE RELEASE INSTEAD
 Text Notes 6100 5950 2    50   ~ 0
@@
 	5400 1550 7450 1550
 $Comp
-L Device:R_US R?
+L Device:R_US R9
 U 1 1 60E31E63
 P 4600 2900
-F 0 "R?" V 4500 3000 50  0000 L CNN
+F 0 "R9" V 4500 3000 50  0000 L CNN
 F 1 "1K" V 4500 2800 50  0000 L CNN
 F 2 "stepper_motor_analyzer:R_0805_2012Metric_Pad1.15x1.40mm_HandSolder" V 4640 2890 50  0001 C CNN
@@
 $EndComp
 $Comp
-L Device:R_US R?
+L Device:R_US R8
 U 1 1 60E32904
 P 4600 1800
-F 0 "R?" V 4500 1900 50  0000 L CNN
+F 0 "R8" V 4500 1900 50  0000 L CNN
 F 1 "1K" V 4500 1700 50  0000 L CNN
 F 2 "stepper_motor_analyzer:R_0805_2012Metric_Pad1.15x1.40mm_HandSolder" V 4640 1790 50  0001 C CNN
@@
 	2900 850  2900 950
 $Comp
-L power:+5V #PWR?
+L power:+5V #PWR0106
 U 1 1 60EA8BA9
 P 2900 850
-F 0 "#PWR?" H 2900 700 50  0001 C CNN
+F 0 "#PWR0106" H 2900 700 50  0001 C CNN
 F 1 "+5V" H 2915 1023 50  0000 C CNN
 F 2 "" H 2900 850 50  0001 C CNN
@@
 	3200 1250 3200 1300
 $Comp
-L Device:R_US R?
+L Device:R_US R7
 U 1 1 60E6D702
 P 3200 1100
-F 0 "R?" H 3300 1150 50  0000 L CNN
+F 0 "R7" H 3300 1150 50  0000 L CNN
 F 1 "1K" H 3300 1050 50  0000 L CNN
 F 2 "stepper_motor_analyzer:R_0805_2012Metric_Pad1.15x1.40mm_HandSolder" V 3240 1090 50  0001 C CNN
@@
 $EndComp
 $Comp
-L Device:R_US R?
+L Device:R_US R6
 U 1 1 60E7C804
 P 2900 1100
-F 0 "R?" H 2700 1150 50  0000 L CNN
+F 0 "R6" H 2700 1150 50  0000 L CNN
 F 1 "DNP" H 2650 1050 50  0000 L CNN
 F 2 "stepper_motor_analyzer:R_0805_2012Metric_Pad1.15x1.40mm_HandSolder" V 2940 1090 50  0001 C CNN

Commit message: Resoted Kicad files to V1.00 release.
Parts:
- removed C4: 1nf, stepper_motor_analyzer:C_0805_2012Metric_Pad1.15x1.40mm_HandSolder, symbol Device:C
- removed C5: DNP, stepper_motor_analyzer:C_0805_2012Metric_Pad1.15x1.40mm_HandSolder, symbol Device:C
- removed R6: DNP, stepper_motor_analyzer:R_0805_2012Metric_Pad1.15x1.40mm_HandSolder, symbol Device:R_US
- removed R7, R8, R9: 1K, stepper_motor_analyzer:R_0805_2012Metric_Pad1.15x1.40mm_HandSolder, symbol Device:R_US
- R4: footprint stepper_motor_analyzer:R_0805_2012Metric_Pad1.15x1.40mm_HandSolder -> stepper_motor_analyzer:R_0805_2012Metric_Pad1.15x1.40mm_HandSolder_no_3d
- U1, U2: value (CURRENT SENSOR) -> ACS70331EOLCTR-2P5B3
Connections:
- net labels removed: +5V, ~TFT_RD
- wire segments 173 -> 157
- no-connect marks 17 -> 20
Other:
- note added: "Simple Stepper Motor Analyzer MK2"
- note removed: "(MK4)"
- note removed: "1K"
- note removed: "1nf"
- note removed: "ACS70331EOLCTR-2P5B3"
- note removed: "ACS712ELCTR-05B-T"
- note removed: "C4, C5"
- note removed: "CONFIG"
- note removed: "DNP"
- note removed: "R4"
- note removed: "R5"
- note removed: "SENSOR"
- note removed: "Simple Stepper Motor Analyzer MK4"
- note removed: "WORK IN PROGRESS. USE RELEASE INSTEAD"
- moved on the sheet: C1, C2, C3, J1, J2, R4, R5, TP3, U1, U2, U3
